File: dual-camera-to-gmsl-serializer-csi-adapter.kicad_sch (KiCad schematic)
At the start: 104 parts, among them J1 Conn_FFC_WE_68715014022, J2 Conn_FFC_WE_68715014022, J3 Conn_FFC_WE_68715014022, U1 TPS2117DRLR, U2 TPS2117DRLR, U3 AP62301_TSOT

Commit message: [#69172] Update PCB
Connections:
- net CAM_RST renamed CAM_FFC_PIN33
- net M1_VSYNC renamed CAM_FFC_PIN32
- net M2_VSYNC renamed CAM_FFC_PIN34
- net M_FREX renamed CAM_FFC_PIN31
Other:
- moved on the sheet: TP1, TP2, TP3, TP4

Commit message: [#69172] Update components
Parts:
- C1: symbol Capacitors0603:C_10u_25V_0603 -> antmicroCapacitors0603:C_10u_25V_0603
- C10, C5, C6, C7, C8, C9: symbol Capacitors0402:C_100n_0402 -> antmicroCapacitors0402:C_100n_0402
- C2: symbol Capacitors0402:C_220n_0402 -> antmicroCapacitors0402:C_220n_0402
- C3, C4: symbol Capacitors0402:C_22u_0402 -> antmicroCapacitors0402:C_22u_0402
- D1, D2, D3, D4, D5, D6: symbol LEDIndicationDiscrete:LED_G_0603_LTST-C190GKT -> antmicroLEDIndicationDiscrete:LED_G_0603_LTST-C190GKT
- H1, H2, H3, H4, H5, H6, H7, H8: symbol MechanicalParts:Spacer_Drill3.7mm_H3mm_9774030151R -> antmicroMechanicalParts:Spacer_Drill3.7mm_H3mm_9774030151R
- J1, J2, J3: symbol FCCConnectors:Conn_FFC_WE_68715014022 -> antmicroFCCConnectors:Conn_FFC_WE_68715014022
- L1: symbol FixedInductors:L_3u3_3.1A_Bourns-SRP3212A -> antmicroFixedInductors:L_3u3_3.1A_Bourns-SRP3212A
- R1, R3, R41: symbol Resistors0402:R_470R_0402 -> antmicroResistors0402:R_470R_0402
- R10, R12, R14, R16, R18, R20, R24, R25, R26, R27, R28, R29, R30, R31, R32, R33, R34, R35, R36, R37, R38, R39, R45, R46, R6, R8: symbol Resistors0402:R_0R_0402 -> antmicroResistors0402:R_0R_0402
- R11, R13, R15, R17, R19, R21, R23, R7, R9: symbol Resistors0402:R_10k_0402 -> antmicroResistors0402:R_10k_0402
- R2, R4, R42: symbol Resistors0402:R_200R_0402 -> antmicroResistors0402:R_200R_0402
- R22: symbol Resistors0402:R_31k6_0402 -> antmicroResistors0402:R_31k6_0402
- R40, R5: symbol Resistors0603:R_0R_22.4A_0603 -> antmicroResistors0603:R_0R_22.4A_0603
- R43, R44: symbol Resistors0402:R_12k_0402 -> antmicroResistors0402:R_12k_0402
- TP1, TP10, TP11, TP12, TP13, TP14, TP15, TP16, TP17, TP18, TP19, TP2, TP20, TP21, TP22, TP23, TP24, TP25, TP26, TP27, TP3, TP4, TP5, TP6, TP7, TP8, TP9: symbol TestPoints:TP_1.5mm_SMD -> antmicroTestPoints:TP_1.5mm_SMD
- U1, U2: symbol PMICPowerDistributionSwitchesLoadDrivers:TPS2117DRLR -> antmicroPMICPowerDistributionSwitchesLoadDrivers:TPS2117DRLR
- U3: symbol DCDCConverters:AP62301_TSOT -> antmicroDCDCConverters:AP62301_TSOT

Commit message: [#69172] Add post-review fixes
Parts:
- removed H1, H2, H3, H4, H5, H6, H7, H8: Spacer_Drill3.7mm_H3mm_9774030151R, antmicro-footprints:Spacer_Drill3.7mm_H3mm_9774030151R, symbol antmicroMechanicalParts:Spacer_Drill3.7mm_H3mm_9774030151R
- removed R11, R13, R15, R17, R19, R21, R7, R9: R_10k_0402, antmicro-footprints:R_0402_1005Metric, symbol antmicroResistors0402:R_10k_0402
- added C11, C13, C15, C17, C18, C21: C_10u_25V_0603, antmicro-footprints:C_0603_1608Metric, symbol antmicroCapacitors0603:C_10u_25V_0603
- added C12, C14, C16, C19, C20, C22: C_100n_0402, antmicro-footprints:C_0402_1005Metric, symbol antmicroCapacitors0402:C_100n_0402
- added H1, H2, H3, H4, H5, H6, H7, H8: Spacer_Drill3.7mm_H6mm_9774060151R, antmicro-footprints:Spacer_Drill3.7mm_H6mm_9774060151R, symbol antmicroMechanicalParts:Spacer_Drill3.7mm_H6mm_9774060151R
- added R11, R13, R15, R17, R19, R21, R7, R9: R_0R_0402, antmicro-footprints:R_0402_1005Metric, symbol antmicroResistors0402:R_0R_0402
- added R47, R48: R_10k_0402, antmicro-footprints:R_0402_1005Metric, symbol antmicroResistors0402:R_10k_0402
- R31, R5: now left out of the parts list
Connections:
- net +5V: now also C11.2, C12.2
- net 3V3_0: now also C17.2, C19.2
- net 3V3_1: now also C18.2, C20.2
- net 3V3_FFC: now also C21.2, C22.2
- net 5V_0: now also C13.2, C14.2
- net 5V_1: now also C15.2, C16.2
- net CAM_FFC_PIN31: now also R19.2, R21.2
- net CAM_FFC_PIN32: now also R15.2, R17.2
- net CAM_FFC_PIN33: now also R11.2, R13.2
- net CAM_FFC_PIN34: now also R7.2, R9.2
- net GND: now also C11.1, C12.1, C13.1, C14.1, C15.1, C16.1, C17.1, C18.1, C19.1, C20.1, C21.1, C22.1, H1.1, H2.1, H3.1, H4.1, H5.1, H6.1, H7.1, H8.1
- net GPIO0_3: now also R43.2, R13.1, R17.1, R21.1, R47.1, R9.1; no longer J2.32, R44.2
- net GPIO1_3: now also R44.2, R11.1, R15.1, R19.1, R48.1, R7.1; no longer J3.32, R43.2
- new net: J3.32, R48.2
- new net: J2.32, R47.2
